File: phonkyo.kicad_sch (KiCad schematic)
At the start: 7 parts, among them J1 GPIO, J2 AudioJack3, U1 CAT24C256

Commit message: finalize rev2 or v0.2
Parts:
- removed J2: AudioJack3, Connector_Audio:Jack_3.5mm_CUI_SJ-3523-SMT_Horizontal, symbol Connector_Audio:AudioJack3
- added C10, C4: 2.2u, Capacitor_SMD:C_0402_1005Metric, symbol Device:C_Small
- added C11, C7: 0.1u, Capacitor_SMD:C_0603_1608Metric, symbol Device:C_Small
- added C12: 0.1u, Capacitor_SMD:C_0402_1005Metric, symbol Device:C_Small
- added C13, C8, C9: 10uf, Capacitor_SMD:C_0603_1608Metric, symbol Device:C_Small
- added C2, C3, C6: 2.2n, Capacitor_SMD:C_0402_1005Metric, symbol Device:C_Small
- added C5: 1u, Capacitor_SMD:C_0603_1608Metric, symbol Device:C_Small
- added J2: LineOutJack, Connector_Audio:Jack_3.5mm_KoreanHropartsElec_PJ-320D-4A_Horizontal, symbol Connector_Audio:AudioJack4
- added J4: RIJack, Connector_Audio:Jack_3.5mm_KoreanHropartsElec_PJ-320D-4A_Horizontal, symbol Connector_Audio:AudioJack4
- added JP2: open, Jumper:SolderJumper-2_P1.3mm_Open_RoundedPad1.0x1.5mm, symbol Jumper:Jumper_2_Small_Open
- added R10, R7, R8, R9: 22, Resistor_SMD:R_0402_1005Metric, symbol Device:R_Small
- added R11: 0, Resistor_SMD:R_0402_1005Metric, symbol Device:R
- added R3, R4: 470, Resistor_SMD:R_0402_1005Metric, symbol Device:R_Small
- added R5: 10k, Resistor_SMD:R_0402_1005Metric, symbol Device:R
- added R6: 20k, Resistor_SMD:R_0402_1005Metric, symbol Device:R
- added U2: PCM5102A, Package_SO:TSSOP-20_4.4x6.5mm_P0.65mm, symbol Audio:PCM5102A
- added U3: XC6206P332MR, Package_TO_SOT_SMD:SOT-23-3, symbol Regulator_Linear:XC6206PxxxMR
Connections:
- net +3V3: now also C11.1, C9.2, U2.20 (DVDD)
- net +5V: now also C5.2, R5.1, U3.3 (VI)
- net GND: now also C11.2, C12.2, C13.1, C6.1, C9.1, J4.R1, J4.R2, J4.S, JP2.1 (A), R11.2, R6.2, U2.10 (DEMP), U2.11 (FLT), U2.16 (FMT), U2.19 (DGND)
- net GPIO18/PCM.CLK: now also R9.1
- net GPIO19/PCM.FS: now also R7.1
- net GPIO21/PCM.DOUT: now also R8.1
- net GPIO25: now also J4.T
- new net: C2.1, J2.R1, R4.1
- new net: R4.2, U2.7 (OUTR)
- new net: R7.2, U2.15 (LRCK)
- new net: C3.2, J2.T, R3.2
- new net: C10.1, U2.5 (VNEG)
- new net: C4.1, U2.4 (CAPM)
- new net: C4.2, U2.2 (CAPP)
- new net: R9.2, U2.13 (BCK)
- new net: C6.2, R5.2, R6.1, U2.17 (XSMT)
- new net: R8.2, U2.14 (DIN)
- new net: JP2.2 (B), R10.1
- new net: R3.1, U2.6 (OUTL)
- new net: R10.2, U2.12 (SCK)
- new net: C12.1, C13.2, U2.18 (LDOO)
- new net +3.3VA: C7.2, C8.2, U2.1 (CPVDD), U2.8 (AVDD), U3.2 (VO)
- new net GNDA: C10.2, C2.2, C3.1, C5.1, C7.1, C8.1, J2.R2, J2.S, R11.1, U2.3 (CPGND), U2.9 (AGND), U3.1 (GND)
Other:
- note added: "Note 1"
- note added: "Note 2"
- company: (none) -> Obcecado

Commit message: finish BOM for v0.2 and submit to production
Parts:
- C1, JP1, JP2, R1, R2, U1: now left out of the parts list
- C12: footprint Capacitor_SMD:C_0402_1005Metric -> Capacitor_SMD:C_0603_1608Metric
Changed lines of the file:
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@@
 		(at 67.31 177.8 0)
 		(unit 1)
-		(exclude_from_sim no)
-		(in_bom yes)
+		(exclude_from_sim yes)
+		(in_bom no)
 		(on_board no)
 		(dnp yes)
@@
 		(at 93.98 170.18 0)
 		(unit 1)
-		(exclude_from_sim no)
-		(in_bom yes)
+		(exclude_from_sim yes)
+		(in_bom no)
 		(on_board no)
 		(dnp yes)
@@
 		(at 96.52 180.34 0)
 		(unit 1)
-		(exclude_from_sim no)
-		(in_bom yes)
+		(exclude_from_sim yes)
+		(in_bom no)
 		(on_board no)
 		(dnp yes)
@@
 		(at 101.6 170.18 0)
 		(unit 1)
-		(exclude_from_sim no)
-		(in_bom yes)
+		(exclude_from_sim yes)
+		(in_bom no)
 		(on_board no)
 		(dnp yes)
@@
 		(at 101.6 162.56 0)
 		(unit 1)
-		(exclude_from_sim no)
-		(in_bom yes)
+		(exclude_from_sim yes)
+		(in_bom no)
 		(on_board no)
 		(dnp yes)
@@
 		(at 81.28 177.8 0)
 		(unit 1)
-		(exclude_from_sim no)
-		(in_bom yes)
+		(exclude_from_sim yes)
+		(in_bom no)
 		(on_board no)
 		(dnp yes)
@@
 		(unit 1)
 		(exclude_from_sim yes)
-		(in_bom yes)
+		(in_bom no)
 		(on_board yes)
 		(dnp no)
@@
 		(at 81.28 190.5 0)
 		(unit 1)
-		(exclude_from_sim no)
-		(in_bom yes)
+		(exclude_from_sim yes)
+		(in_bom no)
 		(on_board no)
 		(dnp yes)
@@
 		(at 101.6 180.34 270)
 		(unit 1)
-		(exclude_from_sim no)
-		(in_bom yes)
+		(exclude_from_sim yes)
+		(in_bom no)
 		(on_board no)
 		(dnp yes)
@@
 			)
 		)
-		(property "Footprint" "Capacitor_SMD:C_0402_1005Metric"
+		(property "Footprint" "Capacitor_SMD:C_0603_1608Metric"
 			(at 231.14 78.74 0)
 			(effects

Commit message: add: revision 0.3
Parts:
- removed JP2: open, Jumper:SolderJumper-2_P1.3mm_Open_RoundedPad1.0x1.5mm, symbol Jumper:Jumper_2_Small_Open
- removed R10: 22, Resistor_SMD:R_0402_1005Metric, symbol Device:R_Small
Connections:
- net GND: now also U2.12 (SCK)
Other:
- moved on the sheet: C10, C11, C4, C6, C9
