File: phonkyo.kicad_sch (KiCad schematic)
At the start: 30 parts, among them J1 GPIO, J2 LineOutJack, J4 RIJack, U1 CAT24C256, U2 PCM5102A, U3 XC6206P332MR

Commit message: pcb: put C11 on DVDD pin 20 and shorten the LDOO route
C11, the 100 nF decoupling cap on DVDD (pin 20), sat 6.0 mm of track
from its pin. That track was a diagonal from (150, 80.7), because the
area above the right column was taken by C12/C13 (the LDOO caps) and
the LDOO route looped around pins 19 and 20 to reach pin 18.

Re-laid out the right-hand fan-out:

- C11 sits directly above pin 20. Track to the pin: 6.0 mm -> 1.1 mm.
- C12 and C13 move beside C11. LDOO runs straight down beside the pins
  to pin 18, replacing the loop. C12 to pin 18: 9.0 mm -> 3.9 mm.
- Pin 19 (DGND) previously ran right to a via in the middle of that
  area. It now goes under the chip body to a via between the pad rows,
  where the board already has two vias.
- The three cap grounds share a new stitching via just above them.

C11 and C12 change from 0603 to 0402. Values are unchanged (100 nF),
and 0402 has lower inductance, which is the point of decoupling. The
schematic footprint fields are updated to match. C13 (10 uF bulk) stays
0603. The new 0402 footprints are cloned from C4 so they match the
board's existing 0402 parts.

XSMT, LRCK and DIN are untouched.

Semantic diff: 3 footprints changed (C11, C12, C13), none added or
removed, 16 tracks/vias replaced by 12, touching only +3V3, GND and
LDOO. DRC with schematic parity matches the baseline: 0 unconnected,
0 parity errors, no new violations.
Parts:
- C11, C12: footprint Capacitor_SMD:C_0603_1608Metric -> Capacitor_SMD:C_0402_1005Metric
Changed lines of the file:
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@@
 			)
 		)
-		(property "Footprint" "Capacitor_SMD:C_0603_1608Metric"
+		(property "Footprint" "Capacitor_SMD:C_0402_1005Metric"
 			(at 177.8 43.18 0)
 			(hide yes)
@@
 			)
 		)
-		(property "Footprint" "Capacitor_SMD:C_0603_1608Metric"
+		(property "Footprint" "Capacitor_SMD:C_0402_1005Metric"
 			(at 231.14 78.74 0)
 			(hide yes)
