File: phonkyo.kicad_sch (KiCad schematic)
At the start: 31 parts, among them J1 GPIO, J2 LineOutJack, J4 RIJack, U1 CAT24C256, U2 PCM5102A, U3 XC6206P332MR

Commit message: design: replace R11 (0R) with a net tie between GND and GNDA
The v0.2 prototype is quiet with the grounds joined, so the 0 ohm link no
longer needs to be removable. NT1 is a KiCad net tie
(NetTie-2_SMD_Pad0.5mm) in the same spot: a copper bridge with no part to
place. It is excluded from the BOM and the placement file, and its pads
are copper-only (no mask opening, no paste). Connectivity is unchanged:
pin 1 on GNDA, pin 2 on GND.

DRC with parity: 0 unconnected, 0 parity, library warnings only. ERC is
unchanged. Production files are regenerated: 28 placed parts, J1 still
left for hand soldering.

Co-Authored-By: Claude Opus 5.5 <noreply@anthropic.com>
Parts:
- NT1: renamed from R11; value 0 -> NetTie; footprint Resistor_SMD:R_0402_1005Metric -> NetTie:NetTie-2_SMD_Pad0.5mm; symbol Device:R -> Device:NetTie_2; LCSC C17168 -> (none); now left out of the parts list
Other:
- moved on the sheet: NT1
Changed lines of the file:
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@@
 	(wire
 		(pts
+			(xy 223.52 121.92) (xy 224.79 121.92)
+		)
+		(stroke
+			(width 0)
+			(type default)
+		)
+	)
+	(wire
+		(pts
+			(xy 229.87 121.92) (xy 231.14 121.92)
+		)
+		(stroke
+			(width 0)
+			(type default)
+		)
+	)
+	(wire
+		(pts
 			(xy 210.82 120.65) (xy 213.36 120.65)
 		)
@@
 	)
 	(symbol
-		(lib_id "Device:R")
-		(at 227.33 121.92 90)
+		(lib_id "Device:NetTie_2")
+		(at 227.33 121.92 0)
 		(unit 1)
 		(body_style 1)
 		(exclude_from_sim no)
-		(in_bom yes)
+		(in_bom no)
 		(on_board yes)
 		(in_pos_files yes)
 		(dnp no)
 		(fields_autoplaced yes)
-		(property "Reference" "R11"
-			(at 227.33 115.57 90)
+		(property "Reference" "NT1"
+			(at 227.33 119.38 0)
 			(show_name no)
 			(do_not_autoplace no)
@@
 			)
 		)
-		(property "Value" "0"
-			(at 227.33 118.11 90)
+		(property "Value" "NetTie"
+			(at 227.33 124.46 0)
 			(show_name no)
 			(do_not_autoplace no)
@@
 			)
 		)
-		(property "Footprint" "Resistor_SMD:R_0402_1005Metric"
+		(property "Footprint" "NetTie:NetTie-2_SMD_Pad0.5mm"
 			(at 227.33 123.698 90)
 			(hide yes)
@@
 			)
 		)
-		(property "LCSC" "C17168"
-			(at 227.33 121.92 0)
-			(hide yes)
-			(show_name no)
-			(do_not_autoplace no)
-			(effects
-				(font
-					(size 1.27 1.27)
-				)
-			)
-		)
-		(property "Description" "Resistor"
+		(property "Description" "Net tie, 2 pins: joins GND and GNDA"
 			(at 227.33 121.92 0)
 			(hide yes)
@@
 			(project "phonkyo"
 				(path "/e63e39d7-6ac0-4ffd-8aa3-1841a4541b55"
-					(reference "R11")
+					(reference "NT1")
 					(unit 1)
 				)
