File: phonkyo.kicad_sch (KiCad schematic)
At the start: 31 parts, among them J1 GPIO, J2 LineOutJack, J4 RIJack, U1 CAT24C256, U2 PCM5102A, U3 XC6206P332MR

Commit message: pcb: move BCK to F.Cu; ESD clamp and series resistor on RI; PWR_FLAGs
BCK (GPIO18) no longer runs 55 mm on B.Cu. Its top-edge run now sits on
F.Cu above the header (y 70.55), over an unbroken B.Cu ground. It drops
through the header gap at x 155.3 to one via, then takes the existing
short B.Cu path to R9. BCK on B.Cu: 54.8 -> 15.1 mm. Total B.Cu track:
102.5 -> 64.1 mm. The GND pour stays one piece and grows 1715 -> 1734 mm2.

To make room, ID_SCL drops through the header gap east of pin 12, and the
+3V3 hop to the EEPROM comes from a rail via at x 123.6. Their B.Cu
segments stay parallel and do not cross.

RI protection: GPIO25 is split where it passes between the +3V3 and +5V
rails. J4's tip now reaches the Pi through R12 (100 R, C25076), with D1
(ESD5Z5.0T1G, C82044) clamping the jack side to GND. The 5 V standoff
leaves a 5 V receiver unclipped. 100 R keeps the transmit level safe
against the receiver's unknown pull-down and limits current into the GPIO
compared with the direct connection. There was no room at the jack
itself: the skull logo and the jack body surround it.

Schematic: R12 and D1 at J4, PWR_FLAGs on +5V, +3V3, GND and GNDA (ERC's
4 power_pin_not_driven errors are gone), and the leftover DNP flag on
JP1's +3V3 symbol is cleared.

DRC with parity: 0 unconnected, 0 parity, library warnings only. ERC: no
errors. Production files are regenerated: 30 placed parts.

Co-Authored-By: Claude Opus 5.5 <noreply@anthropic.com>
Parts:
- added D1: ESD5Z5.0, Diode_SMD:D_SOD-523, symbol Device:D_Zener_Small
- added R12: 100, Resistor_SMD:R_0402_1005Metric, symbol Device:R_Small
Connections:
- net GND: now also D1.2 (A)
- net GPIO25: now also R12.1; no longer J4.T
- new net: D1.1 (K), J4.T, R12.2
